File: Controller Schematic/111/111.kicad_pcb (KiCad board)
At the start: 2 copper layers, 122 parts, among them J1 Screw_Terminal_01x02, J10 Conn_02x13_Top_Bottom, J11 Conn_02x13_Top_Bottom, J12 Conn_02x05_Top_Bottom, J2 Screw_Terminal_01x03, J3 Screw_Terminal_01x02, J4 DS-201, J5 RJ45, J6 Conn_02x13_Top_Bottom, J7 Conn_02x13_Top_Bottom, J8 Conn_02x13_Top_Bottom, J9 Conn_02x13_Top_Bottom, U1 4N35, U10 4N35, U11 4N35, U12 4N35, U13 4N35, U14 4N35, U15 4N35, U16 4N35, U17 4N35, U18 4N35, U19 4N35, U2 4N35, U20 4N35, U21 4N35, U22 4N35, U23 4N35, U24 4N35, U25 4N35, U26 4N35, U27 4N35, U28 4N35, U3 4N35, U4 4N35, U5 4N35, U6 MCP23S17_SP, U7 4N35, U8 4N35, U9 4N35

Commit message: PCB updated
Parts:
- removed C5: 1uF, 50V, Capacitor_SMD:CP_Elec_4x5.7
- removed D10, D15, D16, D17, D18, D19, D20, D24, D26, D27, D28, D29, D30, D8: BL-LS0805UYC, LED_SMD:LED_0805_2012Metric
- removed R26, R6, R7: 330, Resistor_SMD:R_0805_2012Metric
- removed U6: MCP23S17_SP, Package_DIP:DIP-28_W7.62mm
- removed XA1: Arduino_Uno_Shield, Module:Arduino_UNO_R3_WithMountingHoles
- added *D20: BL-LS0805UYC, LED_SMD:LED_0805_2012Metric, F.Cu at (129.9, 63.8)
- added *D24: BL-LS0805UYC, LED_SMD:LED_0805_2012Metric, F.Cu at (105.5, 68.3)
- added *J2: Screw_Terminal_01x02, TerminalBlock_Phoenix:TerminalBlock_Phoenix_MKDS-1,5-2_1x02_P5.00mm_Horizontal, F.Cu at (22.6, 29.8)
- added *R26: 330, Resistor_SMD:R_0805_2012Metric, F.Cu at (134.0, 63.8)
- added *XA1: Arduino_Uno_Shield, Module:Arduino_UNO_R3_WithMountingHoles, F.Cu at (216.2, 66.3)
- added DS1: WC1602A, Display:WC1602A, F.Cu at (67.1, 18.0)
- added JP1: SolderJumper_2_Bridged, Jumper:SolderJumper-2_P1.3mm_Bridged_RoundedPad1.0x1.5mm, F.Cu at (69.7, 89.2)
- added JP10: SolderJumper_2_Open, Jumper:SolderJumper-2_P1.3mm_Open_Pad1.0x1.5mm, F.Cu at (126.6, 109.0)
- added JP11: SolderJumper_2_Open, Jumper:SolderJumper-2_P1.3mm_Open_Pad1.0x1.5mm, F.Cu at (111.9, 106.9)
- added JP12: SolderJumper_2_Open, Jumper:SolderJumper-2_P1.3mm_Open_Pad1.0x1.5mm, F.Cu at (115.4, 111.5)
- added JP13: SolderJumper_2_Open, Jumper:SolderJumper-2_P1.3mm_Open_Pad1.0x1.5mm, F.Cu at (111.9, 111.5)
- added JP2: SolderJumper_2_Bridged, Jumper:SolderJumper-2_P1.3mm_Bridged_RoundedPad1.0x1.5mm, F.Cu at (99.7, 96.8)
- added JP3: SolderJumper_2_Bridged, Jumper:SolderJumper-2_P1.3mm_Bridged_RoundedPad1.0x1.5mm, F.Cu at (108.3, 99.6)
- added JP4: SolderJumper_2_Bridged, Jumper:SolderJumper-2_P1.3mm_Bridged_RoundedPad1.0x1.5mm, F.Cu at (122.8, 109.0)
- added JP5: SolderJumper_2_Bridged, Jumper:SolderJumper-2_P1.3mm_Bridged_RoundedPad1.0x1.5mm, F.Cu at (108.3, 106.9)
- added JP6: SolderJumper_2_Bridged, Jumper:SolderJumper-2_P1.3mm_Bridged_RoundedPad1.0x1.5mm, F.Cu at (118.0, 109.0)
- added JP7: SolderJumper_2_Bridged, Jumper:SolderJumper-2_P1.3mm_Bridged_RoundedPad1.0x1.5mm, F.Cu at (108.3, 111.5)
- added JP8: SolderJumper_2_Open, Jumper:SolderJumper-2_P1.3mm_Open_Pad1.0x1.5mm, F.Cu at (103.2, 96.8)
- added JP9: SolderJumper_2_Open, Jumper:SolderJumper-2_P1.3mm_Open_Pad1.0x1.5mm, F.Cu at (111.9, 99.6)
- added RV1: R_POT, Potentiometer_THT:Potentiometer_Bourns_3339W_Horizontal, F.Cu at (51.3, 22.9)
- added U2: ESP32_DevKit_V1_DOIT, ESP32_DevKit_V1_DOIT:esp32_devkit_v1_doit, F.Cu at (198.6, 43.2)
- added U3: MCP23S17_SP, Package_DIP:DIP-28_W7.62mm, F.Cu at (54.9, 63.0)
- added U5: MCP23S17_SP, Package_DIP:DIP-28_W7.62mm, F.Cu at (162.3, 62.0)
- *D1: renamed from D1; moved to B.Cu
- *D12: renamed from D12; moved to B.Cu
- *D13: renamed from D13; moved to B.Cu
- *R11: renamed from R11; moved to B.Cu
- *R12: renamed from R12; moved to B.Cu
- *R13: renamed from R13; moved to B.Cu
- *R14: renamed from R14; moved to B.Cu
- *R15: renamed from R15; moved to B.Cu
- *R16: renamed from R16; moved to B.Cu
- moved H4 265.3 mm to (21.3, 150.6), turned to 270 degrees
- moved H2 261.6 mm to (21.3, 18.8), turned to 270 degrees
- moved J2 242.5 mm to (22.6, 117.6), turned to 270 degrees
- moved C4 240.6 mm to (40.4, 39.4), turned to 270 degrees
- moved C7 234.4 mm to (51.3, 95.2), turned to 180 degrees
- moved C1 220.5 mm to (229.8, 60.5)
- moved *U2 216.3 mm to (72.4, 80.5), turned to 270 degrees
- moved *R9 211.0 mm to (74.9, 72.0), turned to 90 degrees
- moved U4 196.4 mm to (80.8, 80.3), turned to 90 degrees
- moved R4 194.2 mm to (79.1, 90.4)
- moved D5 190.4 mm to (78.2, 94.6), turned to 90 degrees
- moved *U16 156.3 mm to (89.2, 80.5), turned to 270 degrees
- moved U12 148.1 mm to (131.1, 80.5), turned to 90 degrees
- moved *R25 147.7 mm to (91.7, 72.0), turned to 270 degrees
- moved *U15 145.8 mm to (97.5, 80.5), turned to 270 degrees
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- renumbered D2 to *D2, D21 to *D21, D22 to *D22, D23 to *D23, D3 to *D3, D4 to *D4, D6 to *D6, D9 to *D9, J1 to *J1, J3 to *J3, R10 to *R10, R2 to *R2, R24 to *R24, R25 to *R25, R3 to *R3, R34 to *R34, R35 to *R35, R36 to *R36, R37 to *R37, R38 to *R38, R39 to *R39, R5 to *R5, R9 to *R9, U15 to *U15, U16 to *U16, U2 to *U2, U23 to *U23, U24 to *U24, U25 to *U25, U26 to *U26, U27 to *U27, U28 to *U28, U3 to *U3, U5 to *U5
Connections:
- net ALARMRST_IN renamed SigIn2
- net Alarm renamed SigOut2
- net Net-(J5-Pad3) renamed S1
- net Net-(J5-Pad4) renamed S2
- net NotReadyIN renamed NotSigOut1IN
- net ZPD_IN renamed SigIn3
- net ZSC_IN renamed SigIn4
- *D1 pad 1: ReadyM1 -> SigOut1M2
- *D1 pad 2: ReadyM2 -> SigOut1M1
- *D12 pad 1: ReadyM3 -> SigOut1M4
- *D12 pad 2: ReadyM4 -> SigOut1M3
- *D13 pad 1: ReadyM5 -> SigOut1M6
- *D13 pad 2: ReadyM6 -> SigOut1M5
- *D3 pad 1: Net-(C1-Pad1) -> 5V
- *D4 pad 1: Net-(D4-Pad1) -> COM
- *D4 pad 2: Net-(D4-Pad2) -> Net-(*D4-Pad2)
- *J1 pad 2: Net-(D4-Pad1) -> Net-(*D4-Pad2)
- *R11 pad 1: ReadyM1 -> SigOut1M1
- *R12 pad 1: ReadyM2 -> SigOut1M2
- *R13 pad 1: ReadyM3 -> SigOut1M3
- *R14 pad 1: ReadyM4 -> SigOut1M4
- *R15 pad 1: ReadyM5 -> SigOut1M5
- *R16 pad 1: ReadyM6 -> SigOut1M6
- *R2 pad 1: Net-(C1-Pad1) -> 5V
- *R24 pad 1: ZPDOUT -> #SigIn3
- *R25 pad 1: ZSCOUT -> #SigIn4
- *R3 pad 1: Net-(D4-Pad2) -> Net-(*D4-Pad2)
- *U3 pad 1: Net-(D4-Pad2) -> Net-(*D4-Pad2)
- *U3 pad 2: Net-(D4-Pad1) -> COM
- C1 pad 1: Net-(C1-Pad1) -> 5V
- H1 pad 1: COM -> Net-(H1-Pad1)
- H2 pad 1: COM -> Net-(H2-Pad1)
- J10 pad 11: SRVON_IN -> SigIn1M5
- J10 pad 21: ReadyM5 -> SigOut1M5
- J11 pad 11: SRVON_IN -> SigIn1M6
- J11 pad 21: ReadyM6 -> SigOut1M6
- J6 pad 11: SRVON_IN -> SigIn1M1
- J6 pad 21: ReadyM1 -> SigOut1M1
- J7 pad 11: SRVON_IN -> SigIn1M2
- J7 pad 21: ReadyM2 -> SigOut1M2
- J8 pad 11: SRVON_IN -> SigIn1M3
- J8 pad 21: ReadyM3 -> SigOut1M3
- J9 pad 11: SRVON_IN -> SigIn1M4
- J9 pad 21: ReadyM4 -> SigOut1M4
- R22 pad 1: SRVONOUT -> #SigIn1
- R23 pad 1: AlarmResetOUT -> #SigIn2
- U12 pad 5: AlarmIN -> SigOut2IN
- U13 pad 5: SRVON_IN -> SigIn1
Routing:
- net DC12: track 0.00 -> 643.3 mm, vias 0 -> 29
- net 5V: track 0.00 -> 446.0 mm, vias 0 -> 10
- net SigOut2: track 0.00 -> 332.8 mm, vias 0 -> 13
- net SigIn2: track 0.00 -> 316.1 mm, vias 0 -> 13
- net SigIn3: track 0.00 -> 299.2 mm, vias 0 -> 13
- net SigIn4: track 0.00 -> 297.4 mm, vias 0 -> 13
- net SCK: track 0.00 -> 259.9 mm, vias 0 -> 6
- net SO: track 0.00 -> 258.8 mm, vias 0 -> 6
- net SI: track 0.00 -> 253.4 mm, vias 0 -> 6
- net CS1: track 0.00 -> 213.6 mm, vias 0 -> 4
- net SigIn1M1: track 0.00 -> 167.1 mm, vias 0 -> 3
- net LCDD3: track 0.00 -> 165.6 mm, vias 0 -> 4
- net LCDD4: track 0.00 -> 163.1 mm, vias 0 -> 4
- net LCDD2: track 0.00 -> 160.9 mm, vias 0 -> 4
- net LCDD5: track 0.00 -> 153.7 mm, vias 0 -> 4
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- added copper zone on B.Cu, net COM
- added copper zone on F.Cu, net COM
- added copper zone on B.Cu, net Earth_Protective
- added copper zone on F.Cu, net Earth_Protective
Other:
- board outline added: 227.1 x 139.4 mm
- net class 12V added: clearance 1, trace_width 1, via_dia 1.5, via_drill 1.2
- net class Default: via_drill 0.5 -> 0.8
- rule trace_min: 0.2 -> 0.1
- rule via_min_size: 0.4 -> 0.2
- board text added: "+"
- board text added: "+12V"
- board text added: "1 - COM 2 - DC12 3 - S1IN 4 - S2IN 5 - S3IN 6 - S4IN 7 - S5IN 8 - S6IN"
- board text added: "12V"
- board text added: "5V"
- board text added: "5V from USB"
- board text added: "6DOF control block"
- board text added: "ADDR 001"
- board text added: "ADR 000"
- board text added: "AGND"
- board text added: "ALARM"
- board text added: "ALARM RESET"
- board text added: "AlarmResetOut"
- board text added: "BTN1IN"
- board text added: "COM"
- board text added: "CS0"
- board text added: "CS1"
- board text added: "DC12"
- board text added: "DIR"
- board text added: "DRIVE 1"
- board text added: "DRIVE 2"
- board text added: "DRIVE 3"
- board text added: "DRIVE 4"
- board text added: "DRIVE 5"
- board text added: "DRIVE 6"
- board text added: "DirM1"
- board text added: "DirM2"
- board text added: "DirM3"
- board text added: "DirM4"
- board text added: "DirM5"
- board text added: "DirM6"
- board text added: "GND"
- board text added: "HALL SENSORS"
- board text added: "OZ"
- board text added: "PA+"
- board text added: "PA-"
- board text added: "PB+"
- board text added: "PB-"
- board text added: "PD+"
- board text added: "PD-"
- board text added: "POWER 12V"
- board text added: "POWER 5V"
- board text added: "PP+"
- board text added: "PP-"
- board text added: "PV"
- board text added: "PZ+"
- board text added: "PZ-"
- board text added: "Panel IN"
- board text added: "PanelLed"
- board text added: "Power 12V"
- board text added: "READY"
- board text added: "S1IN"
- board text added: "S2IN"
- board text added: "S3IN"
- board text added: "S4IN"
- board text added: "S5IN"
- board text added: "S6IN"
- board text added: "SCK"
- board text added: "SI"
- board text added: "SO"
- board text added: "SRV-ON"
- board text added: "SRV-ON OUT"
- board text added: "STEP"
- board text added: "Schematic and PCB design by Yakovlev Yuri <krotos139> https://github.com/krotos139/6DOF-Rotary-Stewart-Motion-Simulator 30.11.2020 ver 1.0 SHUIAK"
- board text added: "SigIN2"
- board text added: "SigIn1"
- board text added: "SigIn3"
- board text added: "SigIn4"
- board text added: "SigOut1"
- board text added: "SigOut2"
- board text added: "SigOut3"
- board text added: "SigOut4"
- board text added: "StepM1"
- board text added: "StepM2"
- board text added: "StepM3"
- board text added: "StepM4"
- board text added: "StepM5"
- board text added: "StepM6"
- board text added: "TOGGLE SWITCH"
- board text added: "The control signal of power supply and ground 9 - DC12~24V 10 - COM Input command signal 6 - SigIn1: SRV-ON 7- SigIn2: alarm reset 21- SigIn3: Zero position deviation 8 - SigIn4: Zero speed clamp Output command signal. 11 - SigOUT1： Servo ready 23 - SigOUT2： Alarm detection 12 - SigOUT3： Positioningcomplete 24 - SigOUT4： Zero speed Instruction pulse input port PV:open collector input power Instru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"
- board text added: "Toggle"
- board text added: "Vref"
- board text added: "ZERO POSITION DEVIATION"
- board text added: "ZERO SPEED CLAMP"
- board text added: "ZPD OUT"
- board text added: "ZSC OUT"
- board text added: "lcdD2"
- board text added: "lcdD3"
- board text added: "lcdD4"
- board text added: "lcdD5"
- board text added: "lcdD6"
- board text added: "lcdD7"

Commit message: PCB was changed
Parts:
- removed *D21: BL-LS0805UYC, LED_SMD:LED_0805_2012Metric
- removed *R34, *R35, *R36, *R37, *R38, *R39: 330, Resistor_SMD:R_0805_2012Metric
- removed *U23, *U24, *U25, *U26, *U27, *U28, U17: 4N35, Package_DIP:SMDIP-6_W9.53mm
- removed the J2 at (22.6, 117.6)
- removed JP10, JP11, JP12, JP13, JP8, JP9: SolderJumper_2_Open, Jumper:SolderJumper-2_P1.3mm_Open_Pad1.0x1.5mm
- removed JP4, JP5, JP6, JP7: SolderJumper_2_Bridged, Jumper:SolderJumper-2_P1.3mm_Bridged_RoundedPad1.0x1.5mm
- removed R22: 100, Resistor_SMD:R_0805_2012Metric
- removed the U13 at (114.3, 80.5)
- added C10: 0.1uF 50V, Capacitor_SMD:C_0805_2012Metric, B.Cu at (184.0, 127.3)
- added C11: 0.1uF 50V, Capacitor_SMD:C_0805_2012Metric, F.Cu at (224.2, 91.9)
- added C12: 0.1uF 50V, Capacitor_SMD:C_0805_2012Metric, B.Cu at (217.0, 127.3)
- added C13: 0.1uF 50V, Capacitor_SMD:C_0805_2012Metric, F.Cu at (191.1, 91.9)
- added C14: 0.1uF 50V, Capacitor_SMD:C_0805_2012Metric, B.Cu at (200.5, 127.3)
- added C16: 0.1uF 50V, Capacitor_SMD:C_0805_2012Metric, B.Cu at (43.4, 42.9)
- added C17: 0.1uF 50V, Capacitor_SMD:C_0805_2012Metric, F.Cu at (151.4, 32.6)
- added C18: 0.1uF 50V, Capacitor_SMD:C_0805_2012Metric, F.Cu at (238.0, 61.1)
- added C2: 0.1uF 50V, Capacitor_SMD:C_0805_2012Metric, F.Cu at (141.4, 91.9)
- added C5: 0.1uF 50V, Capacitor_SMD:C_0805_2012Metric, F.Cu at (53.6, 88.8)
- added C9: 0.1uF 50V, Capacitor_SMD:C_0805_2012Metric, F.Cu at (157.9, 91.9)
- added J1: Screw_Terminal_01x03, TerminalBlock_Phoenix:TerminalBlock_Phoenix_MKDS-1,5-3_1x03_P5.00mm_Horizontal, F.Cu at (35.8, 124.5)
- added U10: 4N35, Package_DIP:SMDIP-6_W9.53mm, F.Cu at (231.6, 80.5)
- *U3: renamed from U3; value MCP23S17_SP -> MCP23SigIn1M17_SP
- C3, C7: value 1uF, 50V -> 0.1uF 50V; footprint Capacitor_SMD:CP_Elec_4x5.7 -> Capacitor_SMD:C_0805_2012Metric
- C4, C6, C8: value 1uF, 50V -> 0.1uF 50V; footprint Capacitor_SMD:CP_Elec_4x5.7 -> Capacitor_SMD:C_0805_2012Metric; moved to B.Cu
- JP1: moved to B.Cu
- JP2, JP3: value SolderJumper_2_Bridged -> SolderJumper_2_Open; footprint Jumper:SolderJumper-2_P1.3mm_Bridged_RoundedPad1.0x1.5mm -> Jumper:SolderJumper-2_P1.3mm_Open_Pad1.0x1.5mm; moved to B.Cu
- U3: renamed from U5; value MCP23S17_SP -> MCP23SigIn1M17_SP
- moved C7 156.2 mm to (207.5, 91.9), turned to 0 degrees
- moved C4 128.5 mm to (134.2, 127.3), turned to 180 degrees
- moved C8 68.8 mm to (150.9, 127.3), turned to 180 degrees
- moved C3 59.0 mm to (174.4, 91.9), turned to 0 degrees
- moved JP2 59.0 mm to (139.3, 53.1)
- moved JP3 52.7 mm to (139.3, 56.9)
- moved C6 38.6 mm to (167.5, 127.3), turned to 180 degrees
- moved D2 28.6 mm to (61.7, 113.8)
- moved J2 27.7 mm to (44.9, 113.8)
- moved *D2 22.0 mm to (63.9, 118.6)
- moved *J2 17.7 mm to (54.1, 148.8)
- moved D3 17.5 mm to (92.5, 151.4)
- moved R2 17.5 mm to (92.6, 148.3)
- moved H2 16.2 mm to (36.5, 13.0)
- moved H4 15.2 mm to (36.5, 151.0)
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- renumbered *D4 to *D1, *D24 to *D10, *D20 to *D11, *D9 to *D2, *D6 to *D3, *D3 to *D4, *D1 to *D5, *D12 to *D6, *D13 to *D7, *D22 to *D8, *D23 to *D9, *J3 to *J2, *J2 to *J3, *R3 to *R1, *R16 to *R10, R23 to *R11, *R24 to *R12, *R25 to *R13, *R26 to *R14, R27 to *R15, *R9 to *R2, *R5 to *R3, *R10 to *R4, *R11 to *R5, *R12 to *R6, *R13 to *R7, *R14 to *R8, *R15 to *R9, *U2 to *U1, *U3 to *U2, *U5 to *U4, U14 to *U5, *U15 to *U6, *U16 to *U7, U12 to *U8, C2 to C1, C1 to C15, D5 to D1, D7 to D2, D11 to D3, *D2 to D4, D14 to D5, D25 to D6, J11 to J10, J4 to J2, J5 to J3, J6 to J4, J8 to J5, J10 to J6, J12 to J7, J7 to J8, R4 to R1, R28 to R10, R29 to R11, R30 to R12, R31 to R13, R32 to R14, R33 to R15, R8 to R2, *R2 to R3, R1 to R4, R17 to R5, R18 to R6, R19 to R7, R20 to R8, R21 to R9, U2 to U1, U18 to U11, U19 to U12, U20 to U13, U21 to U14, U22 to U15, U4 to U2, U1 to U4, U7 to U5, U8 to U6, U9 to U7, U10 to U8, U11 to U9
Connections:
- net CS1 renamed CSigIn1M1
- *U1 pad 3: Net-(*U2-Pad3) -> (no net)
- *U1 pad 6: Net-(*U2-Pad6) -> (no net)
- *U2 pad 3: Net-(*U3-Pad3) -> (no net)
- *U2 pad 6: Net-(*U3-Pad6) -> (no net)
- *U3 pad 19: Net-(U3-Pad19) -> (no net)
- *U3 pad 2: #SigIn1 -> (no net)
- *U3 pad 20: Net-(U3-Pad20) -> (no net)
- *U3 pad 23: S1IN -> (no net)
- *U3 pad 24: S2IN -> (no net)
- *U3 pad 25: S3IN -> (no net)
- *U3 pad 26: S4IN -> (no net)
- *U3 pad 27: S5IN -> (no net)
- *U3 pad 28: S6IN -> (no net)
- *U3 pad 3: PanelLED -> #SigIn3
- *U3 pad 4: #SigIn3 -> #SigIn4
- *U3 pad 5: #SigIn4 -> PanelLED
- *U3 pad 6: Net-(U3-Pad6) -> (no net)
- *U3 pad 7: Net-(U3-Pad7) -> (no net)
- *U4 pad 3: Net-(*U5-Pad3) -> (no net)
- *U4 pad 6: Net-(*U5-Pad6) -> (no net)
- *U5 pad 3: Net-(U14-Pad3) -> (no net)
- *U5 pad 6: Net-(U14-Pad6) -> (no net)
- *U6 pad 3: Net-(*U15-Pad3) -> (no net)
- *U6 pad 6: Net-(*U15-Pad6) -> (no net)
- *U7 pad 3: Net-(*U16-Pad3) -> (no net)
- *U7 pad 6: Net-(*U16-Pad6) -> (no net)
- *U8 pad 3: Net-(U12-Pad3) -> (no net)
- *U8 pad 6: Net-(U12-Pad6) -> (no net)
- *XA1 pad 1: Net-(*XA1-Pad1) -> (no net)
- *XA1 pad 10: Net-(*XA1-Pad10) -> /DirM1
- *XA1 pad 11: Net-(*XA1-Pad11) -> /StepM2
- *XA1 pad 12: Net-(*XA1-Pad12) -> /DirM2
- *XA1 pad 13: Net-(*XA1-Pad13) -> /StepM3
- *XA1 pad 14: Net-(*XA1-Pad14) -> /DirM3
- *XA1 pad 15: Net-(*XA1-Pad15) -> (no net)
- *XA1 pad 16: Net-(*XA1-Pad16) -> (no net)
- *XA1 pad 2: Net-(*XA1-Pad2) -> (no net)
- *XA1 pad 23: Net-(*XA1-Pad23) -> (no net)
- *XA1 pad 3: Net-(*XA1-Pad3) -> (no net)
- *XA1 pad 30: Net-(*XA1-Pad30) -> (no net)
- *XA1 pad 31: Net-(*XA1-Pad31) -> (no net)
- *XA1 pad 32: Net-(*XA1-Pad32) -> (no net)
- *XA1 pad 4: Net-(*XA1-Pad4) -> (no net)
- *XA1 pad 8: Net-(*XA1-Pad8) -> (no net)
- *XA1 pad 9: Net-(*XA1-Pad9) -> /StepM1
- C3 pad 1: 5V -> DC12
- C3 pad 2: Earth_Protective -> COM
- C4 pad 1: 5V -> DC12
- C4 pad 2: Earth_Protective -> COM
- DS1 pad 10: Net-(DS1-Pad10) -> (no net)
- DS1 pad 7: Net-(DS1-Pad7) -> (no net)
- DS1 pad 8: Net-(DS1-Pad8) -> (no net)
- DS1 pad 9: Net-(DS1-Pad9) -> (no net)
- H1 pad 1: Net-(H1-Pad1) -> (no net)
- H2 pad 1: Net-(H2-Pad1) -> (no net)
- J10 pad 10: Net-(J11-Pad10) -> (no net)
- J10 pad 12: Net-(J11-Pad12) -> (no net)
- J10 pad 14: Net-(J11-Pad14) -> (no net)
- J10 pad 18: Net-(J11-Pad18) -> (no net)
- J10 pad 22: Net-(J11-Pad22) -> (no net)
- J10 pad 23: Net-(J11-Pad23) -> (no net)
- J10 pad 24: Net-(J11-Pad24) -> (no net)
- J10 pad 25: Net-(J11-Pad25) -> (no net)
- J10 pad 26: Net-(J11-Pad26) -> (no net)
- J10 pad 4: Net-(J11-Pad4) -> (no net)
- J10 pad 5: Net-(J11-Pad5) -> (no net)
- J10 pad 6: Net-(J11-Pad6) -> (no net)
- J10 pad 7: Net-(J11-Pad7) -> (no net)
- J10 pad 8: Net-(J11-Pad8) -> (no net)
- J3 pad 3: S1 -> SigIn1M1
- J3 pad 4: S2 -> SigIn1M2
- J3 pad 5: S3 -> SigIn1M3
- J3 pad 6: S4 -> SigIn1M4
- J3 pad 7: S5 -> SigIn1M5
- J3 pad 8: S6 -> SigIn1M6
- J4 pad 22: SigOut4M1 -> (no net)
- J4 pad 23: SigOut3M1 -> (no net)
- J4 pad 26: Net-(J6-Pad26) -> (no net)
- J4 pad 5: Net-(J6-Pad5) -> (no net)
- J4 pad 7: Net-(J6-Pad7) -> (no net)
- J5 pad 10: Net-(J8-Pad10) -> (no net)
- J5 pad 12: Net-(J8-Pad12) -> (no net)
- J5 pad 14: Net-(J8-Pad14) -> (no net)
- J5 pad 18: Net-(J8-Pad18) -> (no net)
- J5 pad 22: Net-(J8-Pad22) -> (no net)
- J5 pad 23: Net-(J8-Pad23) -> (no net)
- J5 pad 24: Net-(J8-Pad24) -> (no net)
- J5 pad 25: Net-(J8-Pad25) -> (no net)
- J5 pad 26: Net-(J8-Pad26) -> (no net)
- J5 pad 4: Net-(J8-Pad4) -> (no net)
- J5 pad 5: Net-(J8-Pad5) -> (no net)
- J5 pad 6: Net-(J8-Pad6) -> (no net)
- J5 pad 7: Net-(J8-Pad7) -> (no net)
- J5 pad 8: Net-(J8-Pad8) -> (no net)
- J6 pad 10: Net-(J10-Pad10) -> (no net)
- J6 pad 12: Net-(J10-Pad12) -> (no net)
- J6 pad 14: Net-(J10-Pad14) -> (no net)
- J6 pad 18: Net-(J10-Pad18) -> (no net)
- J6 pad 22: Net-(J10-Pad22) -> (no net)
- J6 pad 23: Net-(J10-Pad23) -> (no net)
- J6 pad 24: Net-(J10-Pad24) -> (no net)
- J6 pad 25: Net-(J10-Pad25) -> (no net)
- J6 pad 26: Net-(J10-Pad26) -> (no net)
- J6 pad 4: Net-(J10-Pad4) -> (no net)
- J6 pad 5: Net-(J10-Pad5) -> (no net)
- J6 pad 6: Net-(J10-Pad6) -> (no net)
- J6 pad 7: Net-(J10-Pad7) -> (no net)
- J6 pad 8: Net-(J10-Pad8) -> (no net)
- J8 pad 10: Net-(J7-Pad10) -> (no net)
- J8 pad 12: Net-(J7-Pad12) -> (no net)
- J8 pad 14: Net-(J7-Pad14) -> (no net)
- J8 pad 18: Net-(J7-Pad18) -> (no net)
- J8 pad 22: Net-(J7-Pad22) -> (no net)
- J8 pad 23: Net-(J7-Pad23) -> (no net)
- J8 pad 24: Net-(J7-Pad24) -> (no net)
- J8 pad 25: Net-(J7-Pad25) -> (no net)
- J8 pad 26: Net-(J7-Pad26) -> (no net)
- J8 pad 4: Net-(J7-Pad4) -> (no net)
- J8 pad 5: Net-(J7-Pad5) -> (no net)
- J8 pad 6: Net-(J7-Pad6) -> (no net)
- J8 pad 7: Net-(J7-Pad7) -> (no net)
- J8 pad 8: Net-(J7-Pad8) -> (no net)
- J9 pad 10: Net-(J9-Pad10) -> (no net)
- J9 pad 12: Net-(J9-Pad12) -> (no net)
- J9 pad 14: Net-(J9-Pad14) -> (no net)
- J9 pad 18: Net-(J9-Pad18) -> (no net)
- J9 pad 22: Net-(J9-Pad22) -> (no net)
- J9 pad 23: Net-(J9-Pad23) -> (no net)
- J9 pad 24: Net-(J9-Pad24) -> (no net)
- J9 pad 25: Net-(J9-Pad25) -> (no net)
- J9 pad 26: Net-(J9-Pad26) -> (no net)
- J9 pad 4: Net-(J9-Pad4) -> (no net)
- J9 pad 5: Net-(J9-Pad5) -> (no net)
- J9 pad 6: Net-(J9-Pad6) -> (no net)
- J9 pad 7: Net-(J9-Pad7) -> (no net)
- J9 pad 8: Net-(J9-Pad8) -> (no net)
- JP2 pad 1: SigIn1M1 -> Net-(JP2-Pad1)
- JP2 pad 2: S1 -> PanelLED
- JP3 pad 1: SigIn1M2 -> Net-(JP3-Pad1)
- JP3 pad 2: S2 -> PanelIN
- U1 pad 1: Net-(U2-Pad1) -> (no net)
- U1 pad 10: Net-(U2-Pad10) -> (no net)
- U1 pad 16: Net-(U2-Pad16) -> (no net)
- U1 pad 19: Net-(U2-Pad19) -> (no net)
- U1 pad 2: Net-(U2-Pad2) -> (no net)
- U1 pad 20: Net-(U2-Pad20) -> (no net)
- U1 pad 22: Net-(U2-Pad22) -> (no net)
- U1 pad 23: Net-(U2-Pad23) -> (no net)
- U1 pad 27: Net-(U2-Pad27) -> (no net)
- U1 pad 28: Net-(U2-Pad28) -> (no net)
- U1 pad 3: Net-(U2-Pad3) -> (no net)
- U1 pad 4: Net-(U2-Pad4) -> (no net)
- U1 pad 6: Net-(U2-Pad6) -> (no net)
- U1 pad 7: Net-(U2-Pad7) -> (no net)
- U1 pad 8: Net-(U2-Pad8) -> (no net)
- U1 pad 9: Net-(U2-Pad9) -> (no net)
- U11 pad 3: Net-(U18-Pad3) -> (no net)
- U11 pad 6: Net-(U18-Pad6) -> (no net)
- U12 pad 3: Net-(U19-Pad3) -> (no net)
- U12 pad 6: Net-(U19-Pad6) -> (no net)
- U13 pad 3: Net-(U20-Pad3) -> (no net)
- U13 pad 6: Net-(U20-Pad6) -> (no net)
- U14 pad 3: Net-(U21-Pad3) -> (no net)
- U14 pad 6: Net-(U21-Pad6) -> (no net)
- U15 pad 3: Net-(U22-Pad3) -> (no net)
- U15 pad 6: Net-(U22-Pad6) -> (no net)
- U2 pad 3: Net-(U4-Pad3) -> (no net)
- U2 pad 6: Net-(U4-Pad6) -> (no net)
- U3 pad 19: Net-(U5-Pad19) -> (no net)
- U3 pad 20: Net-(U5-Pad20) -> (no net)
- U3 pad 25: Net-(U5-Pad25) -> Net-(JP2-Pad1)
- U3 pad 26: Net-(U5-Pad26) -> Net-(JP3-Pad1)
- U3 pad 27: Net-(U5-Pad27) -> (no net)
- U4 pad 3: Net-(U1-Pad3) -> (no net)
- U4 pad 6: Net-(U1-Pad6) -> (no net)
- U5 pad 3: Net-(U7-Pad3) -> (no net)
- U5 pad 6: Net-(U7-Pad6) -> (no net)
- U6 pad 3: Net-(U8-Pad3) -> (no net)
- U6 pad 6: Net-(U8-Pad6) -> (no net)
- U7 pad 3: Net-(U9-Pad3) -> (no net)
- U7 pad 6: Net-(U9-Pad6) -> (no net)
- U8 pad 3: Net-(U10-Pad3) -> (no net)
- U8 pad 6: Net-(U10-Pad6) -> (no net)
- U9 pad 3: Net-(U11-Pad3) -> (no net)
- U9 pad 6: Net-(U11-Pad6) -> (no net)
Routing:
- net S3: track 126.2 -> 0.00 mm, vias 2 -> 0
- net S1: track 117.9 -> 0.00 mm, vias 2 -> 0
- net S5: track 114.8 -> 0.00 mm, vias 2 -> 0
- net COM: track 0.00 -> 109.2 mm, vias 15 -> 32
- net S2: track 102.9 -> 0.00 mm, vias 4 -> 0
- net S6: track 97.9 -> 0.00 mm, vias 2 -> 0
- net S4: track 97.1 -> 0.00 mm, vias 2 -> 0
- net SigIn1M3: track 117.6 -> 202.2 mm, vias 3 -> 4
- net SigIn1M1: track 167.1 -> 243.6 mm, vias 3 -> 4
- net SigIn1M4: track 89.1 -> 165.5 mm, vias 3 -> 4
- net #SigIn1: track 72.6 -> 0.00 mm, vias 1 -> 0
- net SigIn1M6: track 42.0 -> 113.3 mm, vias 1 -> 2
- net SigIn1: track 69.7 -> 0.00 mm, vias 4 -> 0
- net PanelIN: track 56.3 -> 125.2 mm, vias 1 -> 3
- net PanelLED: track 33.3 -> 99.0 mm
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Other:
- board size 227.1 x 139.4 mm -> 214.1 x 146.8 mm
- board text added: "Schematic and PCB design by Yakovlev Yuri <krotos139> https://github.com/krotos139/ 6DOF-Rotary-Stewart-Motion-Simulator Date: 30.11.2020 ver 1.0 SHUIAK"
- board text added: "SigIn2"
- board text added: "The control signal of power supply and ground 9 - DC12~24V 10 - COM Input command signal 6 - SigIn1: REF (hall sensor) 7- SigIn2: 21- SigIn3: 8 - SigIn4: Output command signal. 11 - SigOUT1： 23 - SigOUT2： 12 - SigOUT3： 24 - SigOUT4： Instruction pulse input port PV:open collector input power Instruction pulse can be three different ways to input 1：Instruction direction and pulse input 2： Clockwise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"
- board text removed: "ALARM"
- board text removed: "ALARM RESET"
- board text removed: "READY"
- board text removed: "SRV-ON"
- board text removed: "Schematic and PCB design by Yakovlev Yuri <krotos139> https://github.com/krotos139/6DOF-Rotary-Stewart-Motion-Simulator 30.11.2020 ver 1.0 SHUIAK"
- board text removed: "The control signal of power supply and ground 9 - DC12~24V 10 - COM Input command signal 6 - SigIn1: SRV-ON 7- SigIn2: alarm reset 21- SigIn3: Zero position deviation 8 - SigIn4: Zero speed clamp Output command signal. 11 - SigOUT1： Servo ready 23 - SigOUT2： Alarm detection 12 - SigOUT3： Positioningcomplete 24 - SigOUT4： Zero speed Instruction pulse input port PV:open collector input power Instru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"
- board text removed: "ZERO POSITION DEVIATION"
- board text removed: "ZERO SPEED CLAMP"
