File: Controller Schematic/111/111.sch (KiCad schematic (older format))
At the start: 122 parts, among them J1 Screw_Terminal_01x02, J10 Conn_02x13_Top_Bottom, J11 Conn_02x13_Top_Bottom, J12 Conn_02x05_Top_Bottom, J2 Screw_Terminal_01x03, J3 Screw_Terminal_01x02, J4 DS-201, J5 RJ45, J6 Conn_02x13_Top_Bottom, J7 Conn_02x13_Top_Bottom, J8 Conn_02x13_Top_Bottom, J9 Conn_02x13_Top_Bottom, U1 4N35, U10 4N35, U11 4N35, U12 4N35, U13 4N35, U14 4N35, U15 4N35, U16 4N35, U17 4N35, U18 4N35, U19 4N35, U2 4N35, U20 4N35, U21 4N35, U22 4N35, U23 4N35, U24 4N35, U25 4N35, U26 4N35, U27 4N35, U28 4N35, U3 4N35, U4 4N35, U5 4N35, U6 MCP23S17_SP, U7 4N35, U8 4N35, U9 4N35

Commit message: PCB updated
Parts:
- removed C5: 1uF, 50V, Capacitor_SMD:CP_Elec_4x5.7, symbol Device:CP
- removed D10, D15, D16, D17, D18, D19, D26, D27, D28, D29, D30, D8: BL-LS0805UYC, LED_SMD:LED_0805_2012Metric, symbol Device:LED
- removed R6, R7: 330, Resistor_SMD:R_0805_2012Metric, symbol Device:R
- removed U6: MCP23S17_SP, Package_DIP:DIP-28_W7.62mm, symbol Interface_Expansion:MCP23S17_SP
- removed XA1: Arduino_Uno_Shield, Module:Arduino_UNO_R3_WithMountingHoles, symbol MCU_Module:Arduino_UNO_R3
- added *J2: Screw_Terminal_01x02, TerminalBlock_Phoenix:TerminalBlock_Phoenix_MKDS-1,5-2_1x02_P5.00mm_Horizontal, symbol Connector:Screw_Terminal_01x02
- added *XA1: Arduino_Uno_Shield, Module:Arduino_UNO_R3_WithMountingHoles, symbol MCU_Module:Arduino_UNO_R3
- added DS1: WC1602A, Display:WC1602A, symbol Display_Character:WC1602A
- added JP1, JP2, JP3, JP4, JP5, JP6, JP7: SolderJumper_2_Bridged, Jumper:SolderJumper-2_P1.3mm_Bridged_RoundedPad1.0x1.5mm, symbol Jumper:SolderJumper_2_Bridged
- added JP10, JP11, JP12, JP13, JP8, JP9: SolderJumper_2_Open, Jumper:SolderJumper-2_P1.3mm_Open_Pad1.0x1.5mm, symbol Jumper:SolderJumper_2_Open
- added RV1: R_POT, Potentiometer_THT:Potentiometer_Bourns_3339W_Horizontal, symbol Device:R_POT
- added U2: ESP32_DevKit_V1_DOIT, ESP32_DevKit_V1_DOIT:esp32_devkit_v1_doit, symbol ESP32_DevKit_V1_DOIT:ESP32_DevKit_V1_DOIT
- added U3, U5: MCP23S17_SP, Package_DIP:DIP-28_W7.62mm, symbol Interface_Expansion:MCP23S17_SP
- renumbered D1 to *D1, D12 to *D12, D13 to *D13, D2 to *D2, D20 to *D20, D21 to *D21, D22 to *D22, D23 to *D23, D24 to *D24, D3 to *D3, D4 to *D4, D6 to *D6, D9 to *D9, J1 to *J1, J3 to *J3, R10 to *R10, R11 to *R11, R12 to *R12, R13 to *R13, R14 to *R14, R15 to *R15, R16 to *R16, R2 to *R2, R24 to *R24, R25 to *R25, R26 to *R26, R3 to *R3, R34 to *R34, R35 to *R35, R36 to *R36, R37 to *R37, R38 to *R38, R39 to *R39, R5 to *R5, R9 to *R9, U15 to *U15, U16 to *U16, U2 to *U2, U23 to *U23, U24 to *U24, U25 to *U25, U26 to *U26, U27 to *U27, U28 to *U28, U3 to *U3, U5 to *U5
Connections:
- net 5V: now also *D3.1 (A1), *R2.1, C1.1, *J2.2 (Pin_2), *XA1.5 (+5V), DS1.15 (LED(+)), DS1.2 (VDD), RV1.3, U2.15 (VIN), U3.15 (A0), U3.18 (~RESET~), U3.9 (VDD), U5.18 (~RESET~), U5.9 (VDD)
- net BTN1IN: now also U5.28 (GPA7)
- net COM: now also *D4.1 (K), *U3.2; no longer H1.1, H2.1
- net DC12: now also JP1.1 (A)
- net DirM1: now also U5.7 (GPB6)
- net DirM2: now also U5.8 (GPB7)
- net DirM3: now also U5.21 (GPA0)
- net DirM4: now also U5.22 (GPA1)
- net DirM5: now also U5.23 (GPA2)
- net DirM6: now also U5.24 (GPA3)
- net Earth_Protective: now also *J2.1 (Pin_1), *XA1.29 (GND), *XA1.6 (GND), *XA1.7 (GND), DS1.1 (VSS), DS1.16 (LED(-)), DS1.5 (R/W), RV1.1, U2.14 (GND), U2.17 (GND), U3.10 (VSS), U3.16 (A1), U3.17 (A2), U5.10 (VSS), U5.15 (A0), U5.16 (A1), U5.17 (A2)
- net PanelIN: now also U3.8 (GPB7)
- net PanelLED: now also U3.3 (GPB2)
- net S1IN: now also U3.23 (GPA2)
- net S2IN: now also U3.24 (GPA3)
- net S3: now also JP4.2 (B)
- net S3IN: now also U3.25 (GPA4)
- net S4: now also JP5.2 (B)
- net S4IN: now also U3.26 (GPA5)
- net S5: now also JP6.2 (B)
- net S5IN: now also U3.27 (GPA6)
- net S6: now also JP7.2 (B)
- net S6IN: now also U3.28 (GPA7)
- net SCK: now also *XA1.28 (D13), U2.11 (IO14), U3.12 (SCK), U5.12 (SCK)
- net SI: now also *XA1.26 (D11), U2.13 (IO13), U3.13 (SI), U5.13 (SI)
- net SO: now also *XA1.27 (D12), U2.12 (IO12), U3.14 (SO), U5.14 (SO)
- net StepM1: now also U5.1 (GPB0)
- net StepM2: now also U5.2 (GPB1)
- net StepM3: now also U5.3 (GPB2)
- net StepM4: now also U5.4 (GPB3)
- net StepM5: now also U5.5 (GPB4)
- net StepM6: now also U5.6 (GPB5)
- net at *U2.4, J2.3 (Pin_3): now also JP1.2 (B)
- net S1: now reaches *U24.2, J5.3
- net S1: now also JP2.2 (B)
- net S2: now reaches *U23.2, J5.4
- net S2: now also JP3.2 (B)
- net at *D4.2 (A), *R3.1, *U3.1: now also *J1.2 (Pin_2)
- net ALARMRST_IN renamed SigIn2
- net Alarm renamed SigOut2
- net AlarmIN renamed SigOut2IN
- net SigOut2IN: now also U3.21 (GPA0)
- net AlarmResetOUT renamed #SigIn2
- net #SigIn2: now also U3.1 (GPB0)
- net NotReadyIN renamed NotSigOut1IN
- net NotSigOut1IN: now also U3.22 (GPA1)
- net ReadyM1 renamed SigOut1M1
- net SigOut1M1: now also *D1.2 (A); no longer *D1.1 (A)
- net ReadyM2 renamed SigOut1M2
- net SigOut1M2: now also *D1.1 (A); no longer *D1.2 (A)
- net ReadyM3 renamed SigOut1M3
- net SigOut1M3: now also *D12.2 (A); no longer *D12.1 (A)
- net ReadyM4 renamed SigOut1M4
- net SigOut1M4: now also *D12.1 (A); no longer *D12.2 (A)
- net ReadyM5 renamed SigOut1M5
- net SigOut1M5: now also *D13.2 (A); no longer *D13.1 (A)
- net ReadyM6 renamed SigOut1M6
- net SigOut1M6: now also *D13.1 (A); no longer *D13.2 (A)
- net SRVONOUT renamed #SigIn1
- net #SigIn1: now also U3.2 (GPB1)
- removed net SRVON_IN: J10.11 (Pin_11), J11.11 (Pin_11), J6.11 (Pin_11), J7.11 (Pin_11), J8.11 (Pin_11), J9.11 (Pin_11), U13.5
- net ZPDOUT renamed #SigIn3
- net #SigIn3: now also U3.4 (GPB3)
- net ZPD_IN renamed SigIn3
- net ZSCOUT renamed #SigIn4
- net #SigIn4: now also U3.5 (GPB4)
- net ZSC_IN renamed SigIn4
- new net: DS1.3 (VO), RV1.2
- new net CS0: *XA1.25 (D10), U2.18 (IO15), U5.11 (~CS~)
- new net CS1: *XA1.24 (D9), U2.21 (IO16), U3.11 (~CS~)
- new net LCDD2: *XA1.17 (D2), DS1.4 (RS), U2.29 (IO22)
- new net LCDD3: *XA1.18 (D3), DS1.6 (E), U2.26 (IO21)
- new net LCDD4: *XA1.19 (D4), DS1.11 (D4), U2.5 (IO35)
- new net LCDD5: *XA1.20 (D5), DS1.12 (D5), U2.24 (IO18)
- new net LCDD6: *XA1.21 (D6), DS1.13 (D6), U2.30 (IO23)
- new net LCDD7: *XA1.22 (D7), DS1.14 (D7), U2.25 (IO19)
- new net SigIn1: JP10.1 (A), JP11.1 (A), JP12.1 (A), JP13.1 (A), JP8.1 (A), JP9.1 (A), U13.5
- new net SigIn1M1: J6.11 (Pin_11), JP2.1 (A), JP8.2 (B)
- new net SigIn1M2: J7.11 (Pin_11), JP3.1 (A), JP9.2 (B)
- new net SigIn1M3: J8.11 (Pin_11), JP10.2 (B), JP4.1 (A)
- new net SigIn1M4: J9.11 (Pin_11), JP11.2 (B), JP5.1 (A)
- new net SigIn1M5: J10.11 (Pin_11), JP12.2 (B), JP6.1 (A)
- new net SigIn1M6: J11.11 (Pin_11), JP13.2 (B), JP7.1 (A)
Other:
- note added: "Arduino UNO (not installed)"
- note added: "Components marked with an asterisk(*) do not need to be installed"
- note added: "Connectors for each driver"
- note added: "Digital outputs"
- note added: "ESP32 DEV KIT"
- note added: "Hall sensor"
- note added: "I/O Expanders #1"
- note added: "I/O Expanders #2"
- note added: "Jampers"
- note added: "LCD Display"
- note added: "Power supply 5V"
- note added: "SigOut1 signals from drivers"
- note added: "SigOut2 signal from drivers"
- note added: "Steps and Dirs outputs for each driver"
- note added: "button"
- note added: "platform activation toggle switch"
- note added: "power supply 12V"
- moved on the sheet: *D1, *D12, *D13, *D2, *D20, *D21, *D22, *D23, *D24, *D3, *D4, *D6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

Commit message: PCB was changed
Parts:
- removed *D21: BL-LS0805UYC, LED_SMD:LED_0805_2012Metric, symbol Device:LED
- removed *R34, *R35, *R36, *R37, *R38, *R39: 330, Resistor_SMD:R_0805_2012Metric, symbol Device:R
- removed *U23, *U24, *U25, *U26, *U27, *U28, U13: 4N35, Package_DIP:SMDIP-6_W9.53mm, symbol Isolator:4N35
- removed C3, C4, C6, C7, C8: 1uF, 50V, Capacitor_SMD:CP_Elec_4x5.7, symbol Device:CP
- removed JP10, JP11, JP12, JP13, JP8, JP9: SolderJumper_2_Open, Jumper:SolderJumper-2_P1.3mm_Open_Pad1.0x1.5mm, symbol Jumper:SolderJumper_2_Open
- removed JP2, JP3, JP4, JP5, JP6, JP7: SolderJumper_2_Bridged, Jumper:SolderJumper-2_P1.3mm_Bridged_RoundedPad1.0x1.5mm, symbol Jumper:SolderJumper_2_Bridged
- removed R22: 100, Resistor_SMD:R_0805_2012Metric, symbol Device:R
- added C10, C11, C12, C13, C14, C16, C17, C18, C2, C3, C4, C5, C6, C7, C8, C9: 0.1uF 50V, Capacitor_SMD:C_0805_2012Metric, symbol Device:C
- added JP2, JP3: SolderJumper_2_Open, Jumper:SolderJumper-2_P1.3mm_Open_Pad1.0x1.5mm, symbol Jumper:SolderJumper_2_Open
- *U3: renamed from U3; value MCP23S17_SP -> MCP23SigIn1M17_SP
- U3: renamed from U5; value MCP23S17_SP -> MCP23SigIn1M17_SP
- renumbered *D4 to *D1, *D24 to *D10, *D20 to *D11, *D9 to *D2, *D6 to *D3, *D3 to *D4, *D1 to *D5, *D12 to *D6, *D13 to *D7, *D22 to *D8, *D23 to *D9, *J3 to *J2, *J2 to *J3, *R3 to *R1, *R16 to *R10, R23 to *R11, *R24 to *R12, *R25 to *R13, *R26 to *R14, R27 to *R15, *R9 to *R2, *R5 to *R3, *R10 to *R4, *R11 to *R5, *R12 to *R6, *R13 to *R7, *R14 to *R8, *R15 to *R9, *U2 to *U1, *U3 to *U2, *U5 to *U4, U14 to *U5, *U15 to *U6, *U16 to *U7, U12 to *U8, C2 to C1, C1 to C15, D5 to D1, D7 to D2, D11 to D3, *D2 to D4, D14 to D5, D25 to D6, J2 to J1, J11 to J10, J4 to J2, J5 to J3, J6 to J4, J8 to J5, J10 to J6, J12 to J7, J7 to J8, R4 to R1, R28 to R10, R29 to R11, R30 to R12, R31 to R13, R32 to R14, R33 to R15, R8 to R2, *R2 to R3, R1 to R4, R17 to R5, R18 to R6, R19 to R7, R20 to R8, R21 to R9, U2 to U1, U17 to U10, U18 to U11, U19 to U12, U20 to U13, U21 to U14, U22 to U15, U4 to U2, U1 to U4, U7 to U5, U8 to U6, U9 to U7, U10 to U8, U11 to U9
Connections:
- net S1 is gone; now on net SigIn1M1: J3.3
- net S2 is gone; now on net SigIn1M2: J3.4
- net S3 is gone; now on net SigIn1M3: J3.5
- net S4 is gone; now on net SigIn1M4: J3.6
- net S5 is gone; now on net SigIn1M5: J3.7
- net S6 is gone; now on net SigIn1M6: J3.8
- net #SigIn3: now also *U3.3 (GPB2); no longer *U3.4 (GPB3)
- net #SigIn4: now also *U3.4 (GPB3); no longer *U3.5 (GPB4)
- net 5V: now also C16.1, C17.1, C18.1
- net COM: now also C10.2, C11.2, C12.2, C13.2, C14.2, C2.2, C3.2, C4.2, C5.2, C6.2, C7.2, C8.2, C9.2
- net DC12: now also C10.1, C11.1, C12.1, C13.1, C14.1, C2.1, C3.1, C4.1, C5.1, C6.1, C7.1, C8.1, C9.1
- net DirM1: now also *XA1.10 (A1)
- net DirM2: now also *XA1.12 (A3)
- net DirM3: now also *XA1.14 (SCL/A5)
- net Earth_Protective: now also C16.2, C17.2, C18.2
- net PanelIN: now also JP3.2 (B)
- net PanelLED: now also *U3.5 (GPB4), JP2.2 (B); no longer *U3.3 (GPB2)
- net StepM1: now also *XA1.9 (A0)
- net StepM2: now also *XA1.11 (A2)
- net StepM3: now also *XA1.13 (SDA/A4)
- net at U3.25 (GPA4): now also JP2.1 (A)
- net at U3.26 (GPA5): now also JP3.1 (A)
- net CS1 renamed CSigIn1M1
- net S1IN renamed SigIn1M1IN
- net S2IN renamed SigIn1M2IN
- net S3IN renamed SigIn1M3IN
- net S4IN renamed SigIn1M4IN
- net S5IN renamed SigIn1M5IN
- net S6IN renamed SigIn1M6IN
Other:
- note removed: "Jampers"
- moved on the sheet: *D11, *R14, *R15, *U8, *XA1
