File: Pedals/Pedals.kicad_pcb (KiCad board)
At the start: 2 copper layers, 62.2 x 50.8 mm, 25 parts, among them J1 Conn_01x06, J2 Screw_Terminal_01x03, J3 Screw_Terminal_01x03, J4 Screw_Terminal_01x03, J5 DB9_Male_MountingHoles, J6 Conn_01x06, J7 Conn_01x04, J8 Conn_01x15, J9 Conn_01x15

Commit message: I've modified Pedal's PCB. I've added gerber files
Parts:
- added LOGO1: Logo_Open_Hardware_Large, Symbol:OSHW-Logo2_14.6x12mm_Copper, B.Cu at (33.0, 67.3)
- C3: value 100uF 25V -> 10uF 25V; footprint Capacitor_SMD:CP_Elec_6.3x7.7 -> Capacitor_SMD:CP_Elec_5x5.4
- C5, C6, C7: moved to B.Cu
- J6: footprint Connector_PinHeader_2.54mm:PinHeader_1x06_P2.54mm_Vertical -> Connector_PinSocket_2.54mm:PinSocket_1x06_P2.54mm_Vertical
- J7: footprint Connector_PinHeader_2.54mm:PinHeader_1x04_P2.54mm_Vertical -> Connector_PinSocket_2.54mm:PinSocket_1x04_P2.54mm_Vertical
- J8, J9: footprint Connector_PinHeader_2.54mm:PinHeader_1x15_P2.54mm_Vertical -> Connector_PinSocket_2.54mm:PinSocket_1x15_P2.54mm_Vertical
- moved J3 44.3 mm to (16.5, 55.9)
- moved J4 44.2 mm to (16.5, 39.4)
- moved R1 39.4 mm to (14.0, 33.9), turned to 270 degrees
- moved D1 37.4 mm to (16.5, 34.0), turned to 90 degrees
- moved H4 25.3 mm to (47.0, 38.7)
- moved C7 19.5 mm to (34.3, 37.1), turned to 270 degrees
- moved C3 19.4 mm to (31.1, 45.9)
- moved C5 15.9 mm to (37.5, 37.1), turned to 270 degrees
- moved C6 12.8 mm to (31.1, 37.1), turned to 270 degrees
- moved H2 12.7 mm to (57.1, 72.4)
- moved J2 10.7 mm to (56.5, 37.9), turned to 90 degrees
- moved C1 10.2 mm to (36.2, 44.1)
- moved J6 8.13 mm to (45.7, 62.7)
- moved J1 8.13 mm to (45.7, 67.3)
- moved J7 8.13 mm to (48.3, 44.5)
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Routing:
- net VCC: track 101.0 -> 120.5 mm, vias 6 -> 0
- net PEDAL_CLUCH: track 41.2 -> 28.1 mm, vias 2 -> 0
- net PEDAL_BREAK: track 94.4 -> 86.0 mm
- net PEDAL_GAS: track 31.6 -> 24.4 mm
- net SCK: track 20.5 -> 26.9 mm
- net DT: track 16.9 -> 23.3 mm
- net Net-(D1-Pad2): track 4.61 -> 2.54 mm
- net GND: vias 0 -> 1
Other:
- board size 62.2 x 50.8 mm -> 49.5 x 50.8 mm
- board text added: "A+"
- board text added: "A-"
- board text added: "ARDUINO NANO"
- board text added: "B+"
- board text added: "B-"
- board text added: "BREAK"
- board text added: "CLUCH"
- board text added: "DT"
- board text added: "E+"
- board text added: "E-"
- board text added: "GAS"
- board text added: "GND"
- board text added: "HX711 BOARD"
- board text added: "PWM"
- board text added: "SCK"
- board text added: "TDD AASD servo MMOS pedals ver 1.0"
- board text added: "VCC"
