File: Pedals/Pedals.sch (KiCad schematic (older format))
At the start: 25 parts, among them J1 Conn_01x06, J2 Screw_Terminal_01x03, J3 Screw_Terminal_01x03, J4 Screw_Terminal_01x03, J5 DB9_Male_MountingHoles, J6 Conn_01x06, J7 Conn_01x04, J8 Conn_01x15, J9 Conn_01x15

Commit message: I've modified Pedal's PCB. I've added gerber files
Parts:
- added LOGO1: Logo_Open_Hardware_Large, Symbol:OSHW-Logo2_14.6x12mm_Copper, symbol Graphic:Logo_Open_Hardware_Large
- C3: value 100uF 25V -> 10uF 25V; footprint Capacitor_SMD:CP_Elec_6.3x7.7 -> Capacitor_SMD:CP_Elec_5x5.4
- J6: footprint Connector_PinHeader_2.54mm:PinHeader_1x06_P2.54mm_Vertical -> Connector_PinSocket_2.54mm:PinSocket_1x06_P2.54mm_Vertical
- J7: footprint Connector_PinHeader_2.54mm:PinHeader_1x04_P2.54mm_Vertical -> Connector_PinSocket_2.54mm:PinSocket_1x04_P2.54mm_Vertical
- J8, J9: footprint Connector_PinHeader_2.54mm:PinHeader_1x15_P2.54mm_Vertical -> Connector_PinSocket_2.54mm:PinSocket_1x15_P2.54mm_Vertical
Changed lines of the file:
@@
 F 0 "J6" H 1380 1042 50  0000 L CNN
 F 1 "Conn_01x06" H 1380 951 50  0000 L CNN
-F 2 "Connector_PinHeader_2.54mm:PinHeader_1x06_P2.54mm_Vertical" H 1300 1050 50  0001 C CNN
+F 2 "Connector_PinSocket_2.54mm:PinSocket_1x06_P2.54mm_Vertical" H 1300 1050 50  0001 C CNN
 F 3 "~" H 1300 1050 50  0001 C CNN
 	1    1300 1050
@@
 F 0 "J7" H 1868 1267 50  0000 C CNN
 F 1 "Conn_01x04" H 1868 1176 50  0000 C CNN
-F 2 "Connector_PinHeader_2.54mm:PinHeader_1x04_P2.54mm_Vertical" H 1950 950 50  0001 C CNN
+F 2 "Connector_PinSocket_2.54mm:PinSocket_1x04_P2.54mm_Vertical" H 1950 950 50  0001 C CNN
 F 3 "~" H 1950 950 50  0001 C CNN
 	1    1950 950
@@
 F 0 "J8" H 3580 1592 50  0000 L CNN
 F 1 "Conn_01x15" H 3580 1501 50  0000 L CNN
-F 2 "Connector_PinHeader_2.54mm:PinHeader_1x15_P2.54mm_Vertical" H 3500 1550 50  0001 C CNN
+F 2 "Connector_PinSocket_2.54mm:PinSocket_1x15_P2.54mm_Vertical" H 3500 1550 50  0001 C CNN
 F 3 "~" H 3500 1550 50  0001 C CNN
 	1    3500 1550
@@
 F 0 "J9" H 4218 2467 50  0000 C CNN
 F 1 "Conn_01x15" H 4218 2376 50  0000 C CNN
-F 2 "Connector_PinHeader_2.54mm:PinHeader_1x15_P2.54mm_Vertical" H 4300 1550 50  0001 C CNN
+F 2 "Connector_PinSocket_2.54mm:PinSocket_1x15_P2.54mm_Vertical" H 4300 1550 50  0001 C CNN
 F 3 "~" H 4300 1550 50  0001 C CNN
 	1    4300 1550
@@
 P 2700 2800
 F 0 "C3" H 2818 2846 50  0000 L CNN
-F 1 "100uF 25V" H 2818 2755 50  0000 L CNN
-F 2 "Capacitor_SMD:CP_Elec_6.3x7.7" H 2738 2650 50  0001 C CNN
+F 1 "10uF 25V" H 2818 2755 50  0000 L CNN
+F 2 "Capacitor_SMD:CP_Elec_5x5.4" H 2738 2650 50  0001 C CNN
 F 3 "https://www.chipdip.ru/product0/9000565736" H 2700 2800 50  0001 C CNN
 	1    2700 2800
@@
 $EndComp
 $Comp
-L Graphic:Logo_Open_Hardware_Large #LOGO1
-U 1 1 600440E4
-P 3300 3650
-F 0 "#LOGO1" H 3300 4150 50  0001 C CNN
-F 1 "Logo_Open_Hardware_Large" H 3300 3250 50  0001 C CNN
-F 2 "" H 3300 3650 50  0001 C CNN
-F 3 "~" H 3300 3650 50  0001 C CNN
-	1    3300 3650
-	1    0    0    -1
-$EndComp
+L Graphic:Logo_Open_Hardware_Large LOGO1
+U 1 1 5FFC0C21
+P 1050 5200
+F 0 "LOGO1" H 1516 5341 50  0000 L CNN
+F 1 "Logo_Open_Hardware_Large" H 1516 5250 50  0000 L CNN
+F 2 "Symbol:OSHW-Logo2_14.6x12mm_Copper" H 1516 5159 50  0000 L CNN
+F 3 "~" H 1050 5200 50  0001 C CNN
+	1    1050 5200
+	1    0    0    -1
+$EndComp
